File: Line Converter.kicad_pcb (KiCad board)
At the start: 2 copper layers, 82.6 x 41.9 mm, 13 parts, among them J1 Phono Out, J2 JAMMA Audio, SW1 Mono_Switch, T1 Transformer_1P_SS_2T, T2 Transformer_1P_SS_2T

Commit message: don't remember :)
Parts:
- moved REF** 3.87 mm to (207.0, 72.4)
- moved REF** 3.81 mm to (207.0, 40.6)
Other:
- board size 82.6 x 41.9 mm -> 77.5 x 41.9 mm
Changed lines of the file:
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@@
   )
   (module MountingHole:MountingHole_2.5mm_Pad_Via (layer F.Cu)
-    (at 210.875825 72.445825)
+    (at 207.01 72.39)
     (descr "Mounting Hole 2.5mm")
     (tags "mounting hole 2.5mm")
@@
   )
   (module MountingHole:MountingHole_2.5mm_Pad_Via (layer F.Cu)
-    (at 210.82 40.64)
+    (at 207.01 40.64)
     (descr "Mounting Hole 2.5mm")
     (tags "mounting hole 2.5mm")
@@
     )
   )
-  (gr_text "Anders Conbere <anders@conbere.org>" (at 198.12 48.26) (layer B.SilkS)
+  (gr_text "Anders Conbere <anders@conbere.org>" (at 186.69 41.91) (layer B.SilkS)
     (effects (font (size 1 1) (thickness 0.15)) (justify mirror))
   )
-  (gr_text "Line Converter: V0.1" (at 205.74 46.99) (layer B.SilkS)
+  (gr_text "Line Converter: V0.1" (at 194.31 39.37) (layer B.SilkS)
     (effects (font (size 1 1) (thickness 0.15)) (justify mirror))
   )
-  (gr_line (start 215.9 35.56) (end 215.9 77.47) (layer Edge.Cuts) (width 0.1))
-  (gr_line (start 133.35 35.56) (end 215.9 35.56) (layer Edge.Cuts) (width 0.1))
+  (gr_line (start 210.82 35.56) (end 210.82 77.47) (layer Edge.Cuts) (width 0.1))
+  (gr_line (start 133.35 35.56) (end 210.82 35.56) (layer Edge.Cuts) (width 0.1))
   (gr_line (start 133.35 77.47) (end 133.35 35.56) (layer Edge.Cuts) (width 0.1))
-  (gr_line (start 215.9 77.47) (end 133.35 77.47) (layer Edge.Cuts) (width 0.1))
+  (gr_line (start 210.82 77.47) (end 133.35 77.47) (layer Edge.Cuts) (width 0.1))
   (segment (start 201.24 52.07) (end 201.32 52.15) (width 0.1524) (layer F.Cu) (net 2))
   (segment (start 192.278 52.07) (end 201.24 52.07) (width 0.1524) (layer F.Cu) (net 2))
@@
     (polygon
       (pts
-        (xy 215.9 77.47) (xy 133.35 77.47) (xy 133.35 35.56) (xy 215.9 35.56)
+        (xy 210.82 77.47) (xy 133.35 77.47) (xy 133.35 35.56) (xy 210.82 35.56)
       )
     )
